Commit message: Estabilidade e navegacao: robo nao capota mais e contorna obstaculos
- URDF: lastro inferior (CoG baixo, robo nao tomba ao encostar em obstaculos),
  rodizio frontal sem atrito, garra sem colisao (so visual; usada no T2),
  rebalanceamento de massas; controlador com aceleracoes mais suaves.
- mission_control: salvaguarda anti-capotamento (IMU); exploracao por campo
  potencial (atracao para o lado inimigo + repulsao dos obstaculos -> contorna
  os cilindros); deteccao de travamento + manobra de escape (recuo firme);
  posicionamento final por area (visao) com LIDAR de seguranca.
- flag_detector: min_blob_area calibrado (deteccao mais estavel).
- Parametros novos (mission_params.yaml) e genoma ampliado p/ a fase evolutiva.
- Launch: spawn parametrizavel (spawn_x/y/z/yaw), headless, use_rviz.

File: description/robot.urdf.xacro (robot description, xacro)
@@ -10,5 +10,5 @@
   <xacro:property name="wheel_ygap" value="0.025"/> <!-- Distancia entre as rodas -->
   <xacro:property name="wheel_zoff" value="0.05"/> <!-- Deslocamento da roda em Z -->
-  <xacro:property name="wheel_xoff" value="0.12"/> <!-- Deslocamento da roda em X -->
+  <xacro:property name="wheel_xoff" value="0.05"/> <!-- Deslocamento da roda em X -->
   <xacro:property name="caster_xoff" value="0.14"/> <!-- Deslocamento do caster em X -->
   <!-- Definição de algumas propriedades inerciais -->
@@ -59,5 +59,5 @@
       </geometry>
     </collision>
-    <xacro:box_inertia m="1" w="${base_width}" d="${base_length}" h="${base_height}"/>
+    <xacro:box_inertia m="3" w="${base_width}" d="${base_length}" h="${base_height}"/>
   </link>
   <!-- Definindo a Base do Robô (base footprint) -->
@@ -69,4 +69,22 @@
     <child link="base_footprint"/>
     <origin xyz="0.0 0.0 ${-(wheel_radius+wheel_zoff)}" rpy="0 0 0"/>
+  </joint>
+  <!-- LASTRO: massa pesada bem baixa (perto do chao) abaixa MUITO o centro de
+       massa, deixando o robo "fundo-pesado" -> nao capota ao encostar em
+       obstaculos. E uma modificacao de estabilidade do grupo. -->
+  <link name="ballast_link">
+    <inertial>
+      <origin xyz="0 0 0" rpy="0 0 0"/>
+      <mass value="8.0"/>
+      <inertia ixx="0.06" ixy="0" ixz="0" iyy="0.06" iyz="0" izz="0.06"/>
+    </inertial>
+    <collision>
+      <geometry><box size="0.20 0.20 0.04"/></geometry>
+    </collision>
+  </link>
+  <joint name="ballast_joint" type="fixed">
+    <parent link="base_link"/>
+    <child link="ballast_link"/>
+    <origin xyz="0 0 -0.12" rpy="0 0 0"/>
   </joint>
   <!-- Definindo as Rodas do Robô -->
@@ -89,5 +107,5 @@
         </geometry>
       </collision>
-      <xacro:cylinder_inertia m="2.5" r="${wheel_radius}" h="${wheel_width}"/>
+      <xacro:cylinder_inertia m="1.0" r="${wheel_radius}" h="${wheel_width}"/>
     </link>
     <joint name="${prefix}_joint" type="continuous">
@@ -123,4 +141,10 @@
     <origin xyz="${caster_xoff} 0.0 ${-(base_height/2)}" rpy="0 0 0"/>
   </joint>
+  <!-- Rodizio frontal SEM ATRITO: esfera de junta fixa que desliza. Com atrito
+       alto ela "agarra" em curvas e tomba o robo. mu=0 -> desliza livre. -->
+  <gazebo reference="front_caster">
+    <mu1>0.0</mu1>
+    <mu2>0.0</mu2>
+  </gazebo>
   <!-- Definindo a IMU do Robô (física) -->
   <link name="imu_link">
@@ -483,9 +507,5 @@
       <origin rpy="0 1.57075 0" xyz="0.1 0 0"/>
     </visual>
-    <collision>
-      <geometry>
-        <cylinder length="0.2" radius="0.01"/>
-      </geometry>
-    </collision>
+    <!-- colisao da garra removida (T1): nao fisga o chao -->
     <xacro:cylinder_inertia m="0.01" r="0.01" h="0.2"/>
   </link>
@@ -503,9 +523,5 @@
       </geometry>
     </visual>
-    <collision>
-      <geometry>
-        <box size="0.1 0.02 0.02"/>
-      </geometry>
-    </collision>
+    <!-- colisao da garra removida (T1): nao fisga o chao -->
     <xacro:box_inertia m="0.015" w="0.02" h="0.02" d="0.1"/>
   </link>
@@ -522,10 +538,5 @@
       </geometry>
     </visual>
-    <collision>
-      <origin rpy="0 0 -0.1" xyz="0.03 0 0"/>
-      <geometry>
-        <box size="0.06 0.01 0.01"/>
-      </geometry>
-    </collision>
+    <!-- colisao da garra removida (T1): nao fisga o chao -->
     <xacro:box_inertia m="0.005" w="0.01" h="0.01" d="0.06"/>
   </link>
@@ -544,10 +555,5 @@
       </geometry>
     </visual>
-    <collision>
-      <origin rpy="-3.1415 0 0" xyz="0 0 0"/>
-      <geometry>
-        <box size="0.1 0.02 0.02"/>
-      </geometry>
-    </collision>
+    <!-- colisao da garra removida (T1): nao fisga o chao -->
     <xacro:box_inertia m="0.015" w="0.02" h="0.02" d="0.1"/>
   </link>
@@ -564,10 +570,5 @@
       </geometry>
     </visual>
-    <collision>
-      <origin rpy="0 0 -0.1" xyz="0.03 0 0"/>
-      <geometry>
-        <box size="0.06 0.01 0.01"/>
-      </geometry>
-    </collision>
+    <!-- colisao da garra removida (T1): nao fisga o chao -->
     <xacro:box_inertia m="0.005" w="0.01" h="0.01" d="0.06"/>
   </link>

Commit message: T2: integra a garra do professor e camera RGB para deteccao por cor
- Restaura as colisoes dos bracos e pontas da garra (presentes no robo base
  do professor, removidas no T1) para permitir a captura por atrito, sem
  reintroduzir o tombamento (lastro do T1 mantem a estabilidade).
- Mantem a ordem das juntas do gripper_controller igual a do repositorio base
  (gripper_extension, right_gripper_joint, left_gripper_joint), para que os
  comandos de exemplo do enunciado funcionem como descritos.
- Habilita uma camera RGB comum em /rgb_cam (a deteccao do T2 e por cor,
  bandeira azul RGB 0,73,227) e desativa a camera de segmentacao do T1 para
  aliviar a renderizacao. A segmentacao fica preservada em comentario.
- Troca a ativacao do joint_state_broadcaster por um spawner com novas
  tentativas, em vez de uma chamada unica que falhava com o controller_manager
  lento (headless/VM).

File: description/robot.urdf.xacro (robot description, xacro)
@@ -388,6 +388,8 @@
   </joint>
   <gazebo reference="camera_link">
-    <!-- Insere uma camera comum RGB -->
-    <!-- <sensor name="robot_cam" type="camera">
+    <!-- Camera comum RGB (Trabalho 2): a deteccao por cor usa esta imagem.
+         Publica em /rgb_cam, topico separado da camera de segmentacao para
+         nao haver conflito. A bandeira azul tem a mascara RGB 0,73,227. -->
+    <sensor name="rgb_cam" type="camera">
       <camera>
         <horizontal_fov>1.57</horizontal_fov>
@@ -395,4 +397,5 @@
           <width>320</width>
           <height>240</height>
+          <format>R8G8B8</format>
         </image>
         <clip>
@@ -404,9 +407,11 @@
       <update_rate>15</update_rate>
       <visualize>true</visualize>
-      <topic>robot_cam</topic>
-      <enable_metrics>true</enable_metrics>
-    </sensor> -->
-    <!-- Insere uma camera com segmentacao semantica -->
-    <sensor name="robot_cam" type="segmentation">
+      <topic>rgb_cam</topic>
+    </sensor>
+    <!-- Camera de segmentacao semantica do T1, desativada no T2: a deteccao
+         passou a ser por cor na camera RGB. Manter as duas cameras ativas
+         dobrava a carga de renderizacao e desestabilizava o simulador. Fica
+         preservada aqui caso seja necessario reativar a segmentacao. -->
+    <!-- <sensor name="robot_cam" type="segmentation">
       <topic>robot_cam</topic>
       <camera>
@@ -425,5 +430,5 @@
       <update_rate>15</update_rate>
       <visualize>true</visualize>
-    </sensor>
+    </sensor> -->
     <!-- Insere uma camera bounding box 2D completo -->
     <!-- <sensor name="full_2d" type="boundingbox_camera">
@@ -523,5 +528,11 @@
       </geometry>
     </visual>
-    <!-- colisao da garra removida (T1): nao fisga o chao -->
+    <!-- Colisao restaurada (T2): superficie de pega da garra para segurar
+         a bandeira por atrito. -->
+    <collision>
+      <geometry>
+        <box size="0.1 0.02 0.02"/>
+      </geometry>
+    </collision>
     <xacro:box_inertia m="0.015" w="0.02" h="0.02" d="0.1"/>
   </link>
@@ -538,5 +549,11 @@
       </geometry>
     </visual>
-    <!-- colisao da garra removida (T1): nao fisga o chao -->
+    <!-- Colisao restaurada (T2): ponta da pinca que toca a bandeira. -->
+    <collision>
+      <origin rpy="0 0 -0.1" xyz="0.03 0 0"/>
+      <geometry>
+        <box size="0.06 0.01 0.01"/>
+      </geometry>
+    </collision>
     <xacro:box_inertia m="0.005" w="0.01" h="0.01" d="0.06"/>
   </link>
@@ -555,5 +572,11 @@
       </geometry>
     </visual>
-    <!-- colisao da garra removida (T1): nao fisga o chao -->
+    <!-- Colisao restaurada (T2): superficie de pega da garra. -->
+    <collision>
+      <origin rpy="-3.1415 0 0" xyz="0 0 0"/>
+      <geometry>
+        <box size="0.1 0.02 0.02"/>
+      </geometry>
+    </collision>
     <xacro:box_inertia m="0.015" w="0.02" h="0.02" d="0.1"/>
   </link>
@@ -570,7 +593,31 @@
       </geometry>
     </visual>
-    <!-- colisao da garra removida (T1): nao fisga o chao -->
+    <!-- Colisao restaurada (T2): ponta da pinca que toca a bandeira. -->
+    <collision>
+      <origin rpy="0 0 -0.1" xyz="0.03 0 0"/>
+      <geometry>
+        <box size="0.06 0.01 0.01"/>
+      </geometry>
+    </collision>
     <xacro:box_inertia m="0.005" w="0.01" h="0.01" d="0.06"/>
   </link>
+  <!-- Atrito alto nas superficies de pega da garra (T2): ajuda a segurar a
+       bandeira por atrito durante o transporte, sem escorregar. -->
+  <gazebo reference="left_gripper">
+    <mu1>2.0</mu1>
+    <mu2>2.0</mu2>
+  </gazebo>
+  <gazebo reference="right_gripper">
+    <mu1>2.0</mu1>
+    <mu2>2.0</mu2>
+  </gazebo>
+  <gazebo reference="left_tip">
+    <mu1>2.0</mu1>
+    <mu2>2.0</mu2>
+  </gazebo>
+  <gazebo reference="right_tip">
+    <mu1>2.0</mu1>
+    <mu2>2.0</mu2>
+  </gazebo>
   <!-- ==================================================================== -->
   <!-- MODIFICACAO DO GRUPO: "farol" sinalizador decorativo no topo do robo. -->
